File: VCDO.kicad_pcb (KiCad board)
At the start: 2 copper layers, 93 parts, among them J1 NOTE CV, J10 PROGRAMMING HEADER, J2 MOD CV, J3 WAVE CV, J4 SUB CV, J5 GLIDE TOGGLE, J6 SUB OUT, J7 TEST HEADER, J8 SYNTH POWER, J9 MAIN OUT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

Commit message: start panel and pcb - edge cuts
Parts:
- added G***: LOGO, Sonosus:vcdopanelholes, F.Cu at (0.00, 0.00)
- added G***: LOGO, Sonosus:vcdopanelsilk, F.Cu at (-58.0, 100.0)
- added G***: LOGO, Sonosus:vcdopanelholes, F.Cu at (-108.0, 0.00)
- added REF**: Kosmo_Panel_Slotted_Mounting_Hole, Sonosus:Kosmo_Panel_Slotted_Mounting_Hole, F.Cu at (-11.0, 3.00)
- added REF**: Kosmo_Pot_Hole, Sonosus:Kosmo_Pot_Hole, F.Cu at (-58.0, 130.0)
- added REF**: Kosmo_Pot_Hole, Sonosus:Kosmo_Pot_Hole, F.Cu at (-33.5, 129.5)
- added REF**: Kosmo_Jack_Hole, Sonosus:Kosmo_Jack_Hole, F.Cu at (-48.0, 155.0)
- added REF**: Kosmo_Jack_Hole, Sonosus:Kosmo_Jack_Hole, F.Cu at (-68.0, 155.0)
- added REF**: Kosmo_Jack_Hole, Sonosus:Kosmo_Jack_Hole, F.Cu at (-88.0, 155.0)
- added REF**: Kosmo_Jack_Hole, Sonosus:Kosmo_Jack_Hole, F.Cu at (-88.0, 178.0)
- added REF**: Kosmo_Jack_Hole, Sonosus:Kosmo_Jack_Hole, F.Cu at (-68.0, 178.0)
- added REF**: Kosmo_Jack_Hole, Sonosus:Kosmo_Jack_Hole, F.Cu at (-48.0, 178.0)
- added REF**: Kosmo_Jack_Hole, Sonosus:Kosmo_Jack_Hole, F.Cu at (-28.0, 178.0)
- added REF**: Kosmo_Panel_Slotted_Mounting_Hole, Sonosus:Kosmo_Panel_Slotted_Mounting_Hole, F.Cu at (-11.0, 197.0)
- added REF**: Kosmo_Panel_Slotted_Mounting_Hole, Sonosus:Kosmo_Panel_Slotted_Mounting_Hole, F.Cu at (-105.0, 197.0)
- added REF**: Kosmo_Panel_Slotted_Mounting_Hole, Sonosus:Kosmo_Panel_Slotted_Mounting_Hole, F.Cu at (-105.0, 3.00)
- added REF**: Kosmo_Pot_Hole, Sonosus:Kosmo_Pot_Hole, F.Cu at (-58.0, 54.5)
- added REF**: Kosmo_Pot_Hole, Sonosus:Kosmo_Pot_Hole, F.Cu at (-33.5, 84.5)
- added REF**: Kosmo_Pot_Hole, Sonosus:Kosmo_Pot_Hole, F.Cu at (-83.5, 84.5)
- added REF**: Kosmo_Pot_Hole, Sonosus:Kosmo_Pot_Hole, F.Cu at (-58.0, 104.5)
- added REF**: Kosmo_Pot_Hole, Sonosus:Kosmo_Pot_Hole, F.Cu at (-83.5, 129.5)
- moved C1 273.4 mm to (281.2, 94.0)
- moved C10 273.4 mm to (344.2, 10.0)
- moved C11 273.4 mm to (358.5, -2.00)
- moved C12 273.4 mm to (358.5, 20.5)
- moved C13 273.4 mm to (365.2, -12.5)
- moved C14 273.4 mm to (365.2, 10.0)
- moved C15 273.4 mm to (366.8, 100.8)
- moved C16 273.4 mm to (375.8, 100.8)
- moved C17 273.4 mm to (393.0, 100.0)
- moved C18 273.4 mm to (399.0, -44.0)
- moved C19 273.4 mm to (402.0, 100.0)
- moved C2 273.4 mm to (281.2, 103.0)
- moved C3 273.4 mm to (292.5, 94.0)
- moved C4 273.4 mm to (292.5, 103.0)
- moved C5 273.4 mm to (300.8, 94.0)
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Other:
- board outline added: 198 x 200 mm

Commit message: move pot
Parts:
- moved RV9 490.9 mm to (50.0, 130.0)
- moved RV11 7.46 mm to (50.0, 54.5)
Changed lines of the file:
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@@
     (add_net WAVE_IN)
+  )
+  (module Sonosus:Potentiometer_Alpha_RD901F-40-00D_centred (layer F.Cu)
+    (at 50 54.5)
+    (descr "Potentiometer, vertical, 9mm, single, http://www.taiwanalpha.com.tw/downloads?target=products&id=113")
+    (tags "potentiometer vertical 9mm single")
+    (fp_text reference RV11 (at 6.45 -4.8 180) (layer F.SilkS)
+      (effects (font (size 1 1) (thickness 0.15)))
+    )
+    (fp_text value "WAVE 10K" (at 0 10.11 180) (layer F.Fab)
+      (effects (font (size 1 1) (thickness 0.15)))
+    )
+    (fp_text user %R (at 7.6524 2.7546) (layer F.Fab)
+      (effects (font (size 1 1) (thickness 0.15)))
+    )
+    (fp_line (start -8.643 6.63) (end 5.107 6.63) (layer F.CrtYd) (width 0.05))
+    (fp_line (start -8.643 -6.71) (end -8.643 6.63) (layer F.CrtYd) (width 0.05))
+    (fp_line (start 5.107 -6.71) (end -8.643 -6.71) (layer F.CrtYd) (width 0.05))
+    (fp_line (start 5.107 6.63) (end 5.107 -6.71) (layer F.CrtYd) (width 0.05))
+    (fp_line (start 4.977 4.83) (end 4.977 -4.91) (layer F.SilkS) (width 0.12))
+    (fp_line (start -6.613 4.83) (end -6.613 3.34) (layer F.SilkS) (width 0.12))
+    (fp_line (start 1.917 4.83) (end 4.977 4.83) (layer F.SilkS) (width 0.12))
+    (fp_line (start -6.613 -4.92) (end -1.893 -4.92) (layer F.SilkS) (width 0.12))
+    (fp_circle (center 0.007 -0.04) (end 0.007 -3.54) (layer F.Fab) (width 0.1))
+    (fp_line (start -6.493 4.71) (end -6.493 -4.79) (layer F.Fab) (width 0.1))
+    (fp_line (start 4.857 4.71) (end 4.857 -4.79) (layer F.Fab) (width 0.1))
+    (fp_line (start -6.493 -4.79) (end 4.857 -4.79) (layer F.Fab) (width 0.1))
+    (fp_line (start -6.493 4.71) (end 4.857 4.71) (layer F.Fab) (width 0.1))
+    (fp_line (start 1.917 -4.91) (end 4.977 -4.91) (layer F.SilkS) (width 0.12))
+    (fp_line (start -6.613 4.83) (end -1.893 4.83) (layer F.SilkS) (width 0.12))
+    (fp_line (start -6.613 -3.73) (end -6.613 -4.91) (layer F.SilkS) (width 0.12))
+    (fp_line (start -6.613 -0.83) (end -6.613 -1.36) (layer F.SilkS) (width 0.12))
+    (fp_line (start -6.613 1.62) (end -6.613 0.79) (layer F.SilkS) (width 0.12))
+    (pad "" thru_hole circle (at 0.007 -4.84 90) (size 3.24 3.24) (drill 1.8) (layers *.Cu *.Mask))
+    (pad "" thru_hole circle (at 0.007 4.76 90) (size 3.24 3.24) (drill 1.8) (layers *.Cu *.Mask))
+    (pad 3 thru_hole circle (at -7.493 2.46 90) (size 1.8 1.8) (drill 1) (layers *.Cu *.Mask)
+      (net 1 GND))
+    (pad 2 thru_hole circle (at -7.493 -0.04 90) (size 1.8 1.8) (drill 1) (layers *.Cu *.Mask)
+      (net 17 WAVEPOT))
+    (pad 1 thru_hole rect (at -7.493 -2.54 90) (size 1.8 1.8) (drill 1) (layers *.Cu *.Mask)
+      (net 2 +5V))
+    (model ${KISYS3DMOD}/Potentiometer_THT.3dshapes/Potentiometer_Alpha_RD901F-40-00D_Single_Vertical.wrl
+      (at (xyz 0 0 0))
+      (scale (xyz 1 1 1))
+      (rotate (xyz 0 0 0))
+    )
   )
   (module Sonosus:vcdopanelholes (layer F.Cu)
@@
   )
   (module Sonosus:Potentiometer_Alpha_RD901F-40-00D_centred (layer F.Cu)
-    (at 49.993 47.04)
-    (descr "Potentiometer, vertical, 9mm, single, http://www.taiwanalpha.com.tw/downloads?target=products&id=113")
-    (tags "potentiometer vertical 9mm single")
-    (fp_text reference RV11 (at 6.45 -4.8 180) (layer F.SilkS)
-      (effects (font (size 1 1) (thickness 0.15)))
-    )
-    (fp_text value "WAVE 10K" (at 0 10.11 180) (layer F.Fab)
-      (effects (font (size 1 1) (thickness 0.15)))
-    )
-    (fp_line (start -8.643 6.63) (end 5.107 6.63) (layer F.CrtYd) (width 0.05))
-    (fp_line (start -8.643 -6.71) (end -8.643 6.63) (layer F.CrtYd) (width 0.05))
-    (fp_line (start 5.107 -6.71) (end -8.643 -6.71) (layer F.CrtYd) (width 0.05))
-    (fp_line (start 5.107 6.63) (end 5.107 -6.71) (layer F.CrtYd) (width 0.05))
-    (fp_line (start 4.977 4.83) (end 4.977 -4.91) (layer F.SilkS) (width 0.12))
-    (fp_line (start -6.613 4.83) (end -6.613 3.34) (layer F.SilkS) (width 0.12))
-    (fp_line (start 1.917 4.83) (end 4.977 4.83) (layer F.SilkS) (width 0.12))
-    (fp_line (start -6.613 -4.92) (end -1.893 -4.92) (layer F.SilkS) (width 0.12))
-    (fp_circle (center 0.007 -0.04) (end 0.007 -3.54) (layer F.Fab) (width 0.1))
-    (fp_line (start -6.493 4.71) (end -6.493 -4.79) (layer F.Fab) (width 0.1))
-    (fp_line (start 4.857 4.71) (end 4.857 -4.79) (layer F.Fab) (width 0.1))
-    (fp_line (start -6.493 -4.79) (end 4.857 -4.79) (layer F.Fab) (width 0.1))
-    (fp_line (start -6.493 4.71) (end 4.857 4.71) (layer F.Fab) (width 0.1))
-    (fp_line (start 1.917 -4.91) (end 4.977 -4.91) (layer F.SilkS) (width 0.12))
-    (fp_line (start -6.613 4.83) (end -1.893 4.83) (layer F.SilkS) (width 0.12))
-    (fp_line (start -6.613 -3.73) (end -6.613 -4.91) (layer F.SilkS) (width 0.12))
-    (fp_line (start -6.613 -0.83) (end -6.613 -1.36) (layer F.SilkS) (width 0.12))
-    (fp_line (start -6.613 1.62) (end -6.613 0.79) (layer F.SilkS) (width 0.12))
-    (fp_text user %R (at 7.6524 2.7546) (layer F.Fab)
-      (effects (font (size 1 1) (thickness 0.15)))
-    )
-    (pad "" thru_hole circle (at 0.007 -4.84 90) (size 3.24 3.24) (drill 1.8) (layers *.Cu *.Mask))
-    (pad "" thru_hole circle (at 0.007 4.76 90) (size 3.24 3.24) (drill 1.8) (layers *.Cu *.Mask))
-    (pad 3 thru_hole circle (at -7.493 2.46 90) (size 1.8 1.8) (drill 1) (layers *.Cu *.Mask)
-      (net 1 GND))
-    (pad 2 thru_hole circle (at -7.493 -0.04 90) (size 1.8 1.8) (drill 1) (layers *.Cu *.Mask)
-      (net 17 WAVEPOT))
-    (pad 1 thru_hole rect (at -7.493 -2.54 90) (size 1.8 1.8) (drill 1) (layers *.Cu *.Mask)
-      (net 2 +5V))
-    (model ${KISYS3DMOD}/Potentiometer_THT.3dshapes/Potentiometer_Alpha_RD901F-40-00D_Single_Vertical.wrl
-      (at (xyz 0 0 0))
-      (scale (xyz 1 1 1))
-      (rotate (xyz 0 0 0))
-    )
-  )
-  (module Sonosus:Potentiometer_Alpha_RD901F-40-00D_centred (layer F.Cu)
     (at 478.5 10)
     (descr "Potentiometer, vertical, 9mm, single, http://www.taiwanalpha.com.tw/downloads?target=products&id=113")
@@
   )
   (module Sonosus:Potentiometer_Alpha_RD901F-40-00D_centred (layer F.Cu)
-    (at 517.662 -19.336)
+    (at 49.993 130.04)
     (descr "Potentiometer, vertical, 9mm, single, http://www.taiwanalpha.com.tw/downloads?target=products&id=113")
     (tags "potentiometer vertical 9mm single")

Commit message: ill do more tomorrow...
Parts:
- moved RV8 443.8 mm to (24.5, 84.5)
- moved RV12 427.0 mm to (74.5, 84.5)
- moved RV9 24.5 mm to (74.5, 129.5)
Other:
- outline, holes or cut-outs redrawn
Changed lines of the file:
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@@
     (pad_to_mask_clearance 0)
     (aux_axis_origin 0 0)
-    (visible_elements 7FFFFFFF)
+    (visible_elements 7FFFF7FF)
     (pcbplotparams
       (layerselection 0x010fc_ffffffff)
@@
   )
   (module Sonosus:Potentiometer_Alpha_RD901F-40-00D_centred (layer F.Cu)
-    (at 495 10)
+    (at 74.5 84.5)
     (descr "Potentiometer, vertical, 9mm, single, http://www.taiwanalpha.com.tw/downloads?target=products&id=113")
     (tags "potentiometer vertical 9mm single")
@@
   )
   (module Sonosus:Potentiometer_Alpha_RD901F-40-00D_centred (layer F.Cu)
-    (at 49.993 130.04)
+    (at 74.5 129.5)
     (descr "Potentiometer, vertical, 9mm, single, http://www.taiwanalpha.com.tw/downloads?target=products&id=113")
     (tags "potentiometer vertical 9mm single")
@@
   )
   (module Sonosus:Potentiometer_Alpha_RD901F-40-00D_centred (layer F.Cu)
-    (at 462 10)
+    (at 24.5 84.5)
     (descr "Potentiometer, vertical, 9mm, single, http://www.taiwanalpha.com.tw/downloads?target=products&id=113")
     (tags "potentiometer vertical 9mm single")
@@
     )
   )
-  (gr_line (start 90 20) (end 90 140) (layer Edge.Cuts) (width 0.1))
-  (gr_line (start 0 20) (end 90 20) (layer Edge.Cuts) (width 0.1))
-  (gr_line (start 0 140) (end 0 20) (layer Edge.Cuts) (width 0.1))
-  (gr_line (start 90 140) (end 0 140) (layer Edge.Cuts) (width 0.1))
+  (gr_line (start 90 35) (end 90 140) (layer Edge.Cuts) (width 0.1))
+  (gr_line (start 5 35) (end 90 35) (layer Edge.Cuts) (width 0.1))
+  (gr_line (start 5 140) (end 5 35) (layer Edge.Cuts) (width 0.1))
+  (gr_line (start 90 140) (end 5 140) (layer Edge.Cuts) (width 0.1))
   (gr_line (start -108 200) (end -108 0) (layer Edge.Cuts) (width 0.05))
   (gr_line (start -8 200) (end -108 200) (layer Edge.Cuts) (width 0.05))

Commit message: import dxf and add 2 pots
Parts:
- added REF**: Kosmo_Pot_Hole, Sonosus:Kosmo_Pot_Hole, F.Cu at (93.8, 40.0)
- added REF**: Kosmo_Pot_Hole, Sonosus:Kosmo_Pot_Hole, F.Cu at (31.2, 40.0)
- moved G*** 213.4 mm to (-210.5, -35.0)
- moved RV11 213.4 mm to (-160.5, 19.5)
- moved RV12 213.4 mm to (-136.0, 49.5)
- moved RV8 213.4 mm to (-186.0, 49.5)
- moved RV9 213.4 mm to (-136.0, 94.5)
Other:
- board size 198 x 200 mm -> 197.5 x 200 mm

Commit message: save
Parts:
- removed the REF** at (93.8, 40.0)
- removed the REF** at (-58.0, 104.5)
- removed the REF** at (-83.5, 129.5)
- removed the REF** at (-58.0, 130.0)
- removed the REF** at (-33.5, 129.5)
- removed the REF** at (-48.0, 155.0)
- removed the REF** at (-68.0, 155.0)
- removed the REF** at (-88.0, 155.0)
- removed the REF** at (-88.0, 178.0)
- removed the REF** at (-68.0, 178.0)
- removed the REF** at (-48.0, 178.0)
- removed the REF** at (31.2, 40.0)
- removed the REF** at (-28.0, 178.0)
- removed the REF** at (-58.0, 54.5)
- removed the REF** at (-33.5, 84.5)
- removed the REF** at (-83.5, 84.5)
- added REF**: Kosmo_Jack_Hole, Sonosus:Kosmo_Jack_Hole, F.Cu at (262.0, 391.0)
- added REF**: Kosmo_Pot_Hole, Sonosus:Kosmo_Pot_Hole, F.Cu at (212.0, 326.0)
- added REF**: Kosmo_Pot_Hole, Sonosus:Kosmo_Pot_Hole, F.Cu at (187.0, 326.0)
- added REF**: Kosmo_Pot_Hole, Sonosus:Kosmo_Pot_Hole, F.Cu at (262.0, 296.0)
- added REF**: Kosmo_Pot_Hole, Sonosus:Kosmo_Pot_Hole, F.Cu at (237.0, 296.0)
- added REF**: Kosmo_Pot_Hole, Sonosus:Kosmo_Pot_Hole, F.Cu at (212.0, 296.0)
- added REF**: Kosmo_Pot_Hole, Sonosus:Kosmo_Pot_Hole, F.Cu at (187.0, 296.0)
- added REF**: Kosmo_Pot_Hole, Sonosus:Kosmo_Pot_Hole, F.Cu at (255.8, 251.0)
- added REF**: Kosmo_Pot_Hole, Sonosus:Kosmo_Pot_Hole, F.Cu at (193.2, 251.0)
- added REF**: Kosmo_Jack_Hole, Sonosus:Kosmo_Jack_Hole, F.Cu at (237.0, 391.0)
- added REF**: Kosmo_Jack_Hole, Sonosus:Kosmo_Jack_Hole, F.Cu at (212.0, 391.0)
- added REF**: Kosmo_Jack_Hole, Sonosus:Kosmo_Jack_Hole, F.Cu at (187.0, 391.0)
- added REF**: Kosmo_Jack_Hole, Sonosus:Kosmo_Jack_Hole, F.Cu at (237.0, 366.0)
- added REF**: Kosmo_Jack_Hole, Sonosus:Kosmo_Jack_Hole, F.Cu at (212.0, 366.0)
- added REF**: Kosmo_Jack_Hole, Sonosus:Kosmo_Jack_Hole, F.Cu at (187.0, 366.0)
- added REF**: Kosmo_Switch_Hole, Sonosus:Kosmo_Switch_Hole, F.Cu at (262.0, 326.0)
- added REF**: Kosmo_Pot_Hole, Sonosus:Kosmo_Pot_Hole, F.Cu at (237.0, 326.0)
- moved REF** 362.7 mm to (284.0, 214.0)
- moved REF** 362.7 mm to (284.0, 408.0)
- moved REF** 342.7 mm to (165.0, 408.0)
- moved REF** 342.7 mm to (165.0, 214.0)
- moved RV8 279.9 mm to (93.8, 40.0)
- moved RV11 192.8 mm to (31.2, 40.0)
Other:
- board size 197.5 x 200 mm -> 125 x 200 mm

Commit message: position pots to panel
Parts:
- moved RV7 440.3 mm to (25.0, 85.0)
- moved RV10 385.9 mm to (100.0, 85.0)
- moved RV1 291.8 mm to (25.0, 115.0)
- moved RV2 257.5 mm to (50.0, 115.0)
- moved RV3 225.3 mm to (75.0, 115.0)
- moved RV12 214.0 mm to (75.0, 85.0)
- moved RV9 186.2 mm to (50.0, 85.0)

Commit message: shufflio
Parts:
- removed G*** (x2): LOGO, Sonosus:vcdopanelholes
- removed G***: LOGO, Sonosus:vcdopanelsilk
- removed REF** (x7): Kosmo_Jack_Hole, Sonosus:Kosmo_Jack_Hole
- removed REF** (x9): Kosmo_Pot_Hole, Sonosus:Kosmo_Pot_Hole
- removed REF** (x4): Kosmo_Panel_Slotted_Mounting_Hole, Sonosus:Kosmo_Panel_Slotted_Mounting_Hole
- removed REF**: Kosmo_Switch_Hole, Sonosus:Kosmo_Switch_Hole
- RV1, RV10, RV11, RV12, RV2, RV3, RV7, RV8, RV9: moved to B.Cu
- moved J1 275.5 mm to (15.8, 132.8)
- moved J2 275.5 mm to (26.2, 132.8)
- moved J3 275.5 mm to (36.0, 132.8)
- moved J4 275.5 mm to (44.2, 132.8)
- moved J5 275.5 mm to (54.8, 132.8)
- moved J6 275.5 mm to (63.8, 133.5)
- moved J9 275.5 mm to (69.8, 133.5)
Other:
- board outline removed

Commit message: edge cuts
Other:
- board outline added: 92 x 89 mm
Changed lines of the file:
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@@
   (general
     (thickness 1.6)
-    (drawings 23)
+    (drawings 27)
     (tracks 0)
     (zones 0)
@@
     (38 B.Mask user)
     (39 F.Mask user)
-    (40 Dwgs.User user)
+    (40 Dwgs.User user hide)
     (41 Cmts.User user)
     (42 Eco1.User user)
@@
     )
   )
+  (gr_line (start 106 33) (end 106 122) (layer Edge.Cuts) (width 0.1))
+  (gr_line (start 14 33) (end 106 33) (layer Edge.Cuts) (width 0.1))
+  (gr_line (start 14 122) (end 14 33) (layer Edge.Cuts) (width 0.1))
+  (gr_line (start 106 122) (end 14 122) (layer Edge.Cuts) (width 0.1))
   (gr_circle (center 50 180) (end 57 180) (layer Dwgs.User) (width 0.2))
   (gr_circle (center 75 180) (end 82 180) (layer Dwgs.User) (width 0.2))
