File: VCDO.kicad_pcb (KiCad board)
At the start: 2 copper layers, 92 x 89 mm, 93 parts, among them J1 NOTE CV, J10 PROGRAMMING HEADER, J2 MOD CV, J3 WAVE CV, J4 SUB CV, J5 GLIDE TOGGLE, J6 SUB OUT, J7 TEST HEADER, J8 SYNTH POWER, J9 MAIN OUT, Q1 2N3904, U1 TL074, U2 TL074, U3 TL072, U4 L7905, U5 L7805, U6 Druid VCDO

Commit message: oops
Other:
- board size 92 x 89 mm -> 100 x 100 mm
Changed lines of the file:
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@@
     (38 B.Mask user)
     (39 F.Mask user)
-    (40 Dwgs.User user hide)
+    (40 Dwgs.User user)
     (41 Cmts.User user)
     (42 Eco1.User user)
@@
     (pad_to_mask_clearance 0)
     (aux_axis_origin 0 0)
-    (visible_elements 7FFFF7FF)
+    (visible_elements 7FFE77FF)
     (pcbplotparams
       (layerselection 0x010fc_ffffffff)
@@
     )
   )
-  (gr_line (start 106 33) (end 106 122) (layer Edge.Cuts) (width 0.1))
-  (gr_line (start 14 33) (end 106 33) (layer Edge.Cuts) (width 0.1))
-  (gr_line (start 14 122) (end 14 33) (layer Edge.Cuts) (width 0.1))
-  (gr_line (start 106 122) (end 14 122) (layer Edge.Cuts) (width 0.1))
+  (gr_line (start 12 33) (end 12 133) (layer Edge.Cuts) (width 0.1))
+  (gr_line (start -88 33) (end 12 33) (layer Edge.Cuts) (width 0.1))
+  (gr_line (start -88 133) (end -88 33) (layer Edge.Cuts) (width 0.1))
+  (gr_line (start 12 133) (end -88 133) (layer Edge.Cuts) (width 0.1))
   (gr_circle (center 50 180) (end 57 180) (layer Dwgs.User) (width 0.2))
   (gr_circle (center 75 180) (end 82 180) (layer Dwgs.User) (width 0.2))

Commit message: add 3d models, sort orientations
Parts:
- 1v/oct: renamed from J1; moved to B.Cu
- C1, C10, C11, C12, C13, C14, C15, C16, C17, C18, C19, C2, C3, C4, C5, C6, C7, C8, C9, D1, D2, D3, D4, D5, D6, D7, D8, J10, J7, J8, JP1, Q1, R1, R10, R11, R12, R13, R14, R15, R16, R17, R18, R19, R2, R20, R21, R22, R23, R24, R25, R26, R27, R28, R29, R3, R30, R31, R32, R33, R34, R35, R36, R4, R5, R6, R7, R8, R9, RV4, RV5, RV6, U1, U2, U3, U4, U5, U6: moved to B.Cu
- FM IN: renamed from J2; moved to B.Cu
- GLIDE SW: renamed from J5; moved to B.Cu
- MAIN OUT: renamed from J9; moved to B.Cu
- RV1, RV10, RV11, RV12, RV2, RV3, RV7, RV8, RV9: moved to F.Cu
- SUB CV: renamed from J4; moved to B.Cu
- SUB OUT: renamed from J6; moved to B.Cu
- WAVE IN: renamed from J3; moved to B.Cu
- moved RV6 253.6 mm to (219.8, 185.0)
- moved R1 232.8 mm to (209.8, 174.0)
- moved R9 232.8 mm to (223.2, 174.0)
- moved C18 228.5 mm to (323.8, 171.8)
- moved Q1 225.7 mm to (260.0, 170.2)
- moved R17 225.7 mm to (254.8, 170.2)
- moved D1 221.4 mm to (235.2, 168.0)
- moved R8 220.0 mm to (214.2, 167.2)
- moved RV5 220.0 mm to (209.8, 167.2)
- moved R13 217.2 mm to (231.5, 165.8)
- moved U1 217.2 mm to (224.8, 165.8)
- moved J10 215.8 mm to (281.0, 165.0)
- moved R20 215.8 mm to (261.5, 165.0)
- moved D2 213.0 mm to (235.2, 163.5)
- moved R36 207.4 mm to (341.0, 160.5)
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
Commit message: save
Parts:
- moved U5 293.2 mm to (30.5, 57.5)
- moved C17 291.1 mm to (27.5, 50.5)
- moved C19 291.1 mm to (36.5, 50.5)
- moved R33 279.8 mm to (29.1, 62.8)
- moved U4 268.2 mm to (30.5, 66.0)
- moved C15 267.8 mm to (27.8, 73.5)
- moved C16 267.8 mm to (36.8, 73.5)
- moved U6 247.6 mm to (81.1, 104.0), turned to 90 degrees
- moved +12 246.3 mm to (15.5, 77.2)
- moved STRIPE 243.7 mm to (15.5, 67.0)
- moved C13 217.9 mm to (89.8, 54.2), turned to 270 degrees
- moved R23 215.2 mm to (82.2, 56.0), turned to 270 degrees
- moved R31 212.9 mm to (108.2, 49.6), turned to 270 degrees
- moved R34 212.1 mm to (108.2, 74.5), turned to 90 degrees
- moved R27 210.9 mm to (101.5, 51.2), turned to 180 degrees
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- renumbered J7 to +12, J8 to STRIPE

Commit message: saveagain
Parts:
- moved C4 118.9 mm to (106.0, 66.8), turned to 270 degrees
- moved R34 7.35 mm to (110.5, 67.5)
- moved C18 4.27 mm to (319.8, 173.2)
- moved C10 1.25 mm to (100.8, 75.5)
- moved C7 1.25 mm to (93.5, 75.5)

Commit message: maybe?
Parts:
- moved C18 5.53 mm to (314.5, 175.0)
Changed lines of the file:
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@@
   )
   (module Sonosus:Capacitor_NonPolarized (layer B.Cu)
-    (at 319.75 173.25)
+    (at 314.5 175)
     (descr "C, Disc series, Radial, pin pitch=5.00mm, , diameter*width=6*4.4mm^2, Capacitor")
     (tags "C Disc series Radial pin pitch 5.00mm  diameter 6mm width 4.4mm Capacitor")

Commit message: sayve
Parts:
- C1, C2, C3, C4, C5, C6: moved to F.Cu
- moved U3 249.1 mm to (61.8, 62.4)
- moved C14 234.2 mm to (61.4, 66.8)
- moved R29 231.6 mm to (69.4, 66.2), turned to 270 degrees
- moved C12 230.9 mm to (57.6, 58.2), turned to 90 degrees
- moved R26 230.9 mm to (58.6, 60.6), turned to 270 degrees
- moved R32 230.3 mm to (79.0, 66.2), turned to 270 degrees
- moved R35 224.8 mm to (91.2, 76.4), turned to 180 degrees
- moved R30 224.6 mm to (75.8, 66.2), turned to 270 degrees
- moved R24 212.3 mm to (72.6, 73.8), turned to 90 degrees
- moved J10 205.7 mm to (78.8, 127.0), turned to 90 degrees
- moved C2 188.7 mm to (33.0, 100.0)
- moved U1 188.4 mm to (46.8, 103.8), turned to 90 degrees
- moved R10 185.7 mm to (46.4, 93.4), turned to 90 degrees
- moved R5 178.3 mm to (45.2, 76.4)
- moved C1 177.9 mm to (40.8, 100.0)
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
Commit message: nearly there
Parts:
- moved R2 187.0 mm to (28.8, 106.6), turned to 180 degrees
- moved C18 125.1 mm to (190.5, 191.6)
- moved JP1 125.1 mm to (217.8, 40.6)
- moved R36 125.1 mm to (217.0, 177.1)
- moved D1 53.9 mm to (182.8, 155.4)
- moved D2 53.9 mm to (182.8, 150.9)
- moved D3 53.9 mm to (182.8, 131.4)
- moved D4 53.9 mm to (182.8, 126.9)
- moved D7 53.9 mm to (182.8, 82.7)
- moved D8 53.9 mm to (182.8, 78.2)
- moved Q1 53.9 mm to (207.6, 157.7)
- moved R1 53.9 mm to (157.3, 161.4)
- moved R12 53.9 mm to (170.8, 88.7)
- moved R13 53.9 mm to (179.1, 153.2)
- moved R14 53.9 mm to (179.1, 129.2)
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
Commit message: almost
Parts:
- C18, R36: moved to F.Cu
- moved R36 172.7 mm to (62.4, 100.2)
- moved RV6 165.6 mm to (17.8, 101.5), turned to 270 degrees
- moved R9 159.9 mm to (25.4, 95.0), turned to 270 degrees
- moved R8 149.0 mm to (22.2, 102.6), turned to 90 degrees
- moved C18 144.5 mm to (78.4, 100.4), turned to 180 degrees
- moved R12 142.0 mm to (30.0, 106.6), turned to 270 degrees
- moved D1 140.9 mm to (56.4, 93.2), turned to 90 degrees
- moved R13 139.3 mm to (53.4, 93.2), turned to 90 degrees
- moved D2 136.5 mm to (59.2, 93.2), turned to 90 degrees
- moved R14 133.2 mm to (50.0, 96.2)
- moved RV5 130.0 mm to (30.9, 124.6)
- moved D3 129.3 mm to (57.6, 99.2), turned to 180 degrees
- moved R7 129.0 mm to (33.2, 114.2), turned to 90 degrees
- moved D4 127.7 mm to (57.6, 102.0), turned to 180 degrees
- moved R1 125.8 mm to (36.6, 126.2), turned to 90 degrees
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Routing:
- added copper zone on F.Cu, net GND
